Commit message: Isaac ROS 3.2

File: hawk_description/urdf/hawk.urdf.xacro (robot description, xacro)
@@ -12,5 +12,5 @@
   <xacro:include filename="$(find hawk_description)/urdf/hawk_macro.urdf.xacro"/>
   <link name="base_link"/>
-  <xacro:hawk_camera name="hawk_stereo" parent="base_link" mount_is_root="true">
+  <xacro:hawk_camera name="hawk_stereo" parent="base_link" mount_is_root="true" add_subsensor_frames="true">
       <origin xyz="0.0 0.0 0.0" rpy="0.0 0.0 0.0"/>
   </xacro:hawk_camera>

File: hawk_description/urdf/hawk_macro.urdf.xacro (robot description, xacro)
@@ -18,7 +18,9 @@
               Default value: base_link
     - mount_is_root: Flag identifying the root link. If true, root is _mount, othewise is _camera.
+    - add_subsensor_frames: Whether to add frames of subs-ensors to the tree (recommended only if
+              driver is not publishing them).
   -->
   <xacro:macro name="hawk_camera" params="*origin name=hawk_stereo parent=base_link
-    mount_is_root:=false">
+    mount_is_root:=false add_subsensor_frames:=false">
     <!-- Constants -->
     <xacro:property name="M_PI" value="3.1415926535897931"/>
@@ -69,37 +71,40 @@
       <child link="${root_link}"/>
     </joint>
-    <!-- Left camera -->
-    <link name="${name}_camera_left"/>
-    <joint name="${name}_camera_left_joint" type="fixed">
-      <origin xyz="0.0 0.0 0.0" rpy="0.0 0.0 0.0"/>
-      <parent link="${name}_camera"/>
-      <child link="${name}_camera_left"/>
-    </joint>
-    <link name="${name}_camera_left_optical"/>
-    <joint name="${name}_camera_left_optical_joint" type="fixed">
-      <origin xyz="0.0 0.0 0.0" rpy="${-M_PI/2} 0.0 ${-M_PI/2}"/>
-      <parent link="${name}_camera_left"/>
-      <child link="${name}_camera_left_optical"/>
-    </joint>
-    <!-- Right camera -->
-    <link name="${name}_camera_right"/>
-    <joint name="${name}_camera_right_joint" type="fixed">
-      <origin xyz="0.0 ${-baseline} 0.0" rpy="0.0 0.0 0.0"/>
-      <parent link="${name}_camera"/>
-      <child link="${name}_camera_right"/>
-    </joint>
-    <link name="${name}_camera_right_optical"/>
-    <joint name="${name}_camera_right_optical_joint" type="fixed">
-      <origin xyz="0.0 0.0 0.0" rpy="${-M_PI/2} 0.0 ${-M_PI/2}"/>
-      <parent link="${name}_camera_right"/>
-      <child link="${name}_camera_right_optical"/>
-    </joint>
-    <!-- IMU -->
-    <link name="${name}_camera_imu"/>
-    <joint name="${name}_camera_imu_joint" type="fixed">
-      <origin xyz="${imu_offset_x} ${imu_offset_y} ${imu_offset_z}" rpy="0.0 ${M_PI/2} 0.0"/>
-      <parent link="${name}_camera"/>
-      <child link="${name}_camera_imu"/>
-    </joint>
+    <!-- Whether to add frames of subs-ensors to the tree (if driver is not publishing them) -->
+    <xacro:if value="${add_subsensor_frames}">
+      <!-- Left camera -->
+      <link name="${name}_camera_left"/>
+      <joint name="${name}_camera_left_joint" type="fixed">
+        <origin xyz="0.0 0.0 0.0" rpy="0.0 0.0 0.0"/>
+        <parent link="${name}_camera"/>
+        <child link="${name}_camera_left"/>
+      </joint>
+      <link name="${name}_camera_left_optical"/>
+      <joint name="${name}_camera_left_optical_joint" type="fixed">
+        <origin xyz="0.0 0.0 0.0" rpy="${-M_PI/2} 0.0 ${-M_PI/2}"/>
+        <parent link="${name}_camera_left"/>
+        <child link="${name}_camera_left_optical"/>
+      </joint>
+      <!-- Right camera -->
+      <link name="${name}_camera_right"/>
+      <joint name="${name}_camera_right_joint" type="fixed">
+        <origin xyz="0.0 ${-baseline} 0.0" rpy="0.0 0.0 0.0"/>
+        <parent link="${name}_camera"/>
+        <child link="${name}_camera_right"/>
+      </joint>
+      <link name="${name}_camera_right_optical"/>
+      <joint name="${name}_camera_right_optical_joint" type="fixed">
+        <origin xyz="0.0 0.0 0.0" rpy="${-M_PI/2} 0.0 ${-M_PI/2}"/>
+        <parent link="${name}_camera_right"/>
+        <child link="${name}_camera_right_optical"/>
+      </joint>
+      <!-- IMU -->
+      <link name="${name}_camera_imu"/>
+      <joint name="${name}_camera_imu_joint" type="fixed">
+        <origin xyz="${imu_offset_x} ${imu_offset_y} ${imu_offset_z}" rpy="0.0 ${M_PI/2} 0.0"/>
+        <parent link="${name}_camera"/>
+        <child link="${name}_camera_imu"/>
+      </joint>
+    </xacro:if>
   </xacro:macro>
 </robot>

File: owl_description/urdf/owl.urdf.xacro (robot description, xacro)
@@ -12,5 +12,5 @@
   <xacro:include filename="$(find owl_description)/urdf/owl_macro.urdf.xacro"/>
   <link name="base_link"/>
-  <xacro:owl_camera name="owl_fisheye" parent="base_link" mount_is_root="true">
+  <xacro:owl_camera name="owl_fisheye" parent="base_link" mount_is_root="true" add_subsensor_frames="true">
       <origin xyz="0.0 0.0 0.0" rpy="0.0 0.0 0.0"/>
   </xacro:owl_camera>

File: owl_description/urdf/owl_macro.urdf.xacro (robot description, xacro)
@@ -17,7 +17,9 @@
     - parent: Parent link where the root of this macro will be connected with a joint.
               Default value: base_link
+    - add_subsensor_frames: Whether to add frames of subs-ensors to the tree (recommended only if
+              driver is not publishing them).
   -->
   <xacro:macro name="owl_camera" params="*origin name=owl_fisheye parent=base_link
-    mount_is_root:=false">
+    mount_is_root:=false add_subsensor_frames:=false">
     <!-- Constants -->
     <xacro:property name="M_PI" value="3.1415926535897931"/>
@@ -64,11 +66,14 @@
       <child link="${root_link}"/>
     </joint>
-    <!-- Optical frame -->
-    <link name="${name}_camera_optical"/>
-    <joint name="${name}_camera_optical_joint" type="fixed">
-        <origin xyz="0.0 0.0 0.0" rpy="${-M_PI/2} 0.0 ${-M_PI/2}"/>
-        <parent link="${name}_camera"/>
-        <child link="${name}_camera_optical"/>
-    </joint>
+    <!-- Whether to add optical frame to the tree (if driver is not publishing it) -->
+    <xacro:if value="${add_subsensor_frames}">
+      <!-- Optical frame -->
+      <link name="${name}_camera_optical"/>
+      <joint name="${name}_camera_optical_joint" type="fixed">
+          <origin xyz="0.0 0.0 0.0" rpy="${-M_PI/2} 0.0 ${-M_PI/2}"/>
+          <parent link="${name}_camera"/>
+          <child link="${name}_camera_optical"/>
+      </joint>
+    </xacro:if>
   </xacro:macro>
 </robot>
